Commit message: Fixed joints

File: body.urdf (robot description, URDF)
Before this commit: robot robot, 3 links, 2 joints
Joints:
- joint Torso_BackLeg: type revolute -> fixed
- joint Torso_FrontLeg: type revolute -> fixed

Commit message: add body

File: body.urdf (robot description, URDF)
Before this commit: robot robot, 3 links, 2 joints
Joints:
- joint Torso_BackLeg: origin xyz=0 1 1 rpy=0 0 0 -> xyz=1 0 1 rpy=0 0 0; type fixed -> revolute
- joint Torso_FrontLeg: origin xyz=0 2 1 rpy=0 0 0 -> xyz=2 0 1 rpy=0 0 0; type fixed -> revolute
